File: tracker/tracker.kicad_sch (KiCad schematic)
At the start: 9 parts, among them U1 XIAO-ESP32-C6-SMD, U2 LIS3DH, U4 INA226AIDGSR

Commit message: started pcb design
Connections:
- net 3v3: now reaches C1.2, C2.2, C3.1, R2.2, R3.1, U1.12 (3V3_OUT), U2.1 (VDD_IO), U2.14 (VDD), U2.8 (CS), U4.6 (VS+)
- net SDA: now reaches R3.2, U1.5 (D4), U2.6 (SDI), U4.4 (SDA)
- net SCL: now reaches R2.1, U1.6 (D5), U2.4 (SPC), U4.5 (SCL)
Other:
- moved on the sheet: C1, C2, C3, R1, R2, R3, U2, U4
