File: tracker_v2/charging_and_battery.kicad_sch (KiCad schematic)
At the start: 17 parts, among them J1 USB_C_Receptacle_PowerOnly_6P, Q1 DMG9926UDM-7, U3 DW01A, U5 TP4056-42-ESOP8

Commit message: completed v2 routing
Parts:
- added TP2, TP7, TP8: TestPoint, TestPoint:TestPoint_Pad_D1.0mm, symbol Connector:TestPoint
Connections:
- net BAT+: now also TP8.1
- net GND: now also TP2.1
- net USB_VBUS: now also TP7.1
