File: tracker_v2/tracker_v2.kicad_sch (KiCad schematic)
At the start: 9 parts, among them U1 XIAO-ESP32-C6-SMD, U2 LIS3DH, U4 INA226AIDGSR

Commit message: completed v2 routing
Parts:
- added TP1, TP3, TP4, TP5, TP6: TestPoint, TestPoint:TestPoint_Pad_D1.0mm, symbol Connector:TestPoint
Connections:
- net 3v3: now also U2.7 (SDO), TP6.1
- net GND: now also TP1.1
- net SCL: now also TP4.1
- net SDA: now also TP3.1
- net at U1.3 (D2), U2.11 (INT1): now also TP5.1
- no-connect marks 21 -> 20
