File: tracker_v3/tracker_v2.kicad_sch (KiCad schematic)
At the start: 16 parts, among them J2 P70-7000045, J3 P70-7000045, U1 XIAO-ESP32-DIP, U2 LIS3DH, U4 INA226AIDGSR

Commit message: added pogo pins to tracker_v3
Parts:
- removed J2, J3: P70-7000045, P70_7000045:HARWIN_P70-7000045, symbol P70-7000045:P70-7000045
- U1: value XIAO-ESP32-DIP -> XIAO-ESP32-C6-SMD; footprint Seeed_Studio_XIAO_Series:XIAO-ESP32-C6-DIP -> Seeed_Studio_XIAO_Series:XIAO-ESP32-C6-SMD
Connections:
- net Shunt_Output: now also U1.23 (VBAT)
- no-connect marks 21 -> 20
