File: tracker_v3/charging_and_battery.kicad_sch (KiCad schematic)
At the start: 20 parts, among them J1 USB_C_Receptacle_PowerOnly_6P, Q1 DMG9926UDM-7, U3 DW01A, U5 TP4056-42-ESOP8

Commit message: v3.0 complete
the v3.0 has been added to cart for buying
Changed lines of the file:
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@@
 		(color 0 0 0 0)
 	)
+	(junction
+		(at 101.6 90.17)
+		(diameter 0)
+		(color 0 0 0 0)
+	)
 	(wire
 		(pts
@@
 	(wire
 		(pts
+			(xy 101.6 104.14) (xy 101.6 90.17)
+		)
+		(stroke
+			(width 0)
+			(type default)
+		)
+	)
+	(wire
+		(pts
 			(xy 55.88 97.79) (xy 55.88 90.17)
 		)
@@
 	(wire
 		(pts
+			(xy 101.6 90.17) (xy 106.68 90.17)
+		)
+		(stroke
+			(width 0)
+			(type default)
+		)
+	)
+	(wire
+		(pts
 			(xy 78.74 113.03) (xy 78.74 134.62)
 		)
@@
 	(wire
 		(pts
-			(xy 111.76 104.14) (xy 123.19 104.14)
-		)
-		(stroke
-			(width 0)
-			(type default)
-		)
-	)
-	(wire
-		(pts
 			(xy 62.23 38.1) (xy 62.23 36.83)
 		)
@@
 	(wire
 		(pts
-			(xy 88.9 90.17) (xy 106.68 90.17)
+			(xy 88.9 90.17) (xy 101.6 90.17)
 		)
 		(stroke
@@
 		)
 		(stroke
+			(width 0)
+			(type default)
+		)
+	)
+	(wire
+		(pts
+			(xy 111.76 104.14) (xy 101.6 104.14)
+		)
+		(stroke
