File: tracker_v3/_restore_backup_2026-10-08T16-11-45-618/tracker_v3.kicad_pcb (KiCad board)
At the start: 2 copper layers, 72.5 x 22.1 mm, 37 parts, among them J1 USB_C_Receptacle_PowerOnly_6P, J2 P70-7000045, J3 P70-7000045, Q1 DMG9926UDM-7, U1 XIAO-ESP32-DIP, U2 LIS3DH, U3 DW01A, U4 INA226AIDGSR, U5 TP4056-42-ESOP8

Commit message: added pogo pins to tracker_v3
Parts:
- removed J2, J3: P70-7000045, P70_7000045:HARWIN_P70-7000045
- removed REF**: Reverb_BTDR-1H, Audio_Module:Reverb_BTDR-1H
- U1: value XIAO-ESP32-DIP -> XIAO-ESP32-C6-SMD
Routing:
- net /Shunt_Output: track 37.7 -> 38.7 mm, vias 2 -> 3
- net GND: track 233.5 -> 234.5 mm, vias 12 -> 13
