File: tracker_v4/tracker_v4.kicad_sch (KiCad schematic)
At the start: 39 parts, among them SW1 SW_Push, SW2 SW_Push, U1 ESP32-C6-MINI-1-N4, U2 LIS3DH, U4 INA226AIDGSR, U5 TPS63020, U7 TPS3899DL01DSER

Commit message: newer version
Parts:
- added R23: 10M, Resistor_SMD:R_0603_1608Metric, symbol Device:R
- L1: value 1.0u -> 1.5u
- R14: value 499k -> 1000k
- R15: value 100k -> 200k
Connections:
- net BUCK_EN: now also R23.2
- net UVLO_SENSE: now also R23.1
Changed lines of the file:
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@@
 	)
 	(junction
+		(at 83.82 146.05)
+		(diameter 0)
+		(color 0 0 0 0)
+	)
+	(junction
 		(at 78.74 74.93)
 		(diameter 0)
@@
 		(color 0 0 0 0)
 	)
+	(junction
+		(at 43.18 153.67)
+		(diameter 0)
+		(color 0 0 0 0)
+	)
 	(no_connect
 		(at 180.34 82.55)
@@
 	(wire
 		(pts
+			(xy 39.37 125.73) (xy 39.37 151.13)
+		)
+		(stroke
+			(width 0)
+			(type default)
+		)
+	)
+	(wire
+		(pts
 			(xy 60.96 59.69) (xy 60.96 48.26)
 		)
@@
 	(wire
 		(pts
+			(xy 39.37 151.13) (xy 43.18 151.13)
+		)
+		(stroke
+			(width 0)
+			(type default)
+		)
+	)
+	(wire
+		(pts
 			(xy 242.57 74.93) (xy 242.57 77.47)
 		)
@@
 	(wire
 		(pts
+			(xy 52.07 125.73) (xy 39.37 125.73)
+		)
+		(stroke
+			(width 0)
+			(type default)
+		)
+	)
+	(wire
+		(pts
 			(xy 134.62 63.5) (xy 140.97 63.5)
 		)
@@
 	(wire
 		(pts
-			(xy 81.28 146.05) (xy 86.36 146.05)
+			(xy 81.28 146.05) (xy 83.82 146.05)
 		)
 		(stroke
@@
 	(wire
 		(pts
+			(xy 59.69 132.08) (xy 83.82 132.08)
+		)
+		(stroke
+			(width 0)
+			(type default)
+		)
+	)
+	(wire
+		(pts
 			(xy 137.16 45.72) (xy 137.16 43.18)
 		)
@@
 	(wire
 		(pts
+			(xy 83.82 132.08) (xy 83.82 146.05)
+		)
+		(stroke
+			(width 0)
+			(type default)
+		)
+	)
+	(wire
+		(pts
 			(xy 21.59 160.02) (xy 21.59 170.18)
 		)
@@
 	(wire
 		(pts
+			(xy 83.82 146.05) (xy 86.36 146.05)
+		)
+		(stroke
+			(width 0)
+			(type default)
+		)
+	)
+	(wire
+		(pts
 			(xy 96.52 45.72) (xy 96.52 49.53)
 		)
@@
 	(wire
 		(pts
+			(xy 43.18 151.13) (xy 43.18 153.67)
+		)
+		(stroke
+			(width 0)
+			(type default)
+		)
+	)
+	(wire
+		(pts
 			(xy 144.78 135.89) (xy 144.78 142.24)
 		)
@@
 	(wire
 		(pts
+			(xy 59.69 125.73) (xy 59.69 132.08)
+		)
+		(stroke
+			(width 0)
+			(type default)
+		)
+	)
+	(wire
+		(pts
 			(xy 116.84 77.47) (xy 116.84 78.74)
 		)
@@
 	(symbol
 		(lib_id "Device:R")
+		(at 55.88 125.73 90)
+		(unit 1)
+		(body_style 1)
+		(exclude_from_sim no)
+		(in_bom yes)
+		(on_board yes)
+		(in_pos_files yes)
+		(dnp no)
+		(fields_autoplaced yes)
+		(property "Reference" "R23"
+			(at 55.88 119.38 90)
+			(show_name no)
+			(do_not_autoplace no)
+			(effects
+				(font
+					(size 1.27 1.27)
+				)
+			)
+		)
+		(property "Value" "10M"
+			(at 55.88 121.92 90)
+			(show_name no)
+			(do_not_autoplace no)
+			(effects
+				(font
+					(size 1.27 1.27)
+				)
+			)
+		)
+		(property "Footprint" "Resistor_SMD:R_0603_1608Metric"
+			(at 55.88 127.508 90)
+			(hide yes)
+			(show_name no)
+			(do_not_autoplace no)
+			(effects
+				(font
+					(size 1.27 1.27)
+				)
+			)
+		)
+		(property "Datasheet" ""
+			(at 55.88 125.73 0)
+			(hide yes)
+			(show_name no)
+			(do_not_autoplace no)
+			(effects
+				(font
+					(size 1.27 1.27)
+				)
+			)
+		)
+		(property "Description" "Resistor"
+			(at 55.88 125.73 0)
+			(hide yes)
+			(show_name no)
+			(do_not_autoplace no)
+			(effects
+				(font
+					(size 1.27 1.27)
+				)
+			)
+		)
+		(pin "2"
+		)
+		(pin "1"
+		)
+		(instances
+			(project "tracker_v4"
+				(path "/0704e846-b6bf-4206-baa8-1088b529855e"
+					(reference "R23")
+					(unit 1)
+				)
+			)
+		)
+	)
+	(symbol
+		(lib_id "Device:R")
 		(at 109.22 39.37 0)
 		(unit 1)
@@
 			)
 		)
-		(property "Value" "100k"
+		(property "Value" "200k"
 			(at 92.71 128.2699 0)
 			(show_name no)
@@
 			)
 		)
-		(property "Value" "1.0u"
+		(property "Value" "1.5u"
 			(at 90.17 55.88 90)
 			(show_name no)
@@
 			)
 		)
-		(property "Value" "499k"
+		(property "Value" "1000k"
 			(at 92.71 115.5699 0)
 			(show_name no)
