File: tracker_v4/charging_and_battery.kicad_sch (KiCad schematic)
At the start: 24 parts, among them J1 USB_C_Receptacle_USB2.0_16P, Q1 DMG9926UDM-7, U3 DW01A, U5 TP4056-42-ESOP8, U6 USBLC6-2SC6

Commit message: corrected schematic
Parts:
- removed D3, D4: D, Diode_SMD:D_SOD-123F, symbol Device:D
- D5: value D -> DO-214AC; footprint Diode_SMD:D_SOD-123F -> Diode_SMD:D_SMA
Connections:
- net GND: now also C5.2, D5.2 (A), R5.2, R6.2; no longer D5.1 (K)
- net USB_DM: no longer J1.A6 (D+), J1.B5 (CC2), J1.B6 (D+), R5.1, U6.1 (I/O1), U6.6 (I/O1)
- net USB_VBUS: now also D5.1 (K)
- new net: J1.B5 (CC2), R5.1
- new net USB_DP: J1.A6 (D+), J1.B6 (D+), U6.1 (I/O1), U6.6 (I/O1)
Other:
- moved on the sheet: R6

Commit message: jk
Parts:
- removed D5: DO-214AC, Diode_SMD:D_SMA, symbol Device:D
- added D3: SMAJ5.0A, Diode_SMD:D_SMA, symbol Diode:SMAJ5.0A
Connections:
- net GND: now also R9.2, D3.2 (A2)
- net PROTECT_MID: no longer R9.2
- net USB_VBUS: now also D3.1 (A1)
Changed lines of the file:
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@@
 	)
 	(junction
-		(at 222.25 118.11)
-		(diameter 0)
-		(color 0 0 0 0)
-	)
-	(junction
 		(at 147.32 81.28)
 		(diameter 0)
@@
 	)
 	(junction
+		(at 180.34 140.97)
+		(diameter 0)
+		(color 0 0 0 0)
+	)
+	(junction
 		(at 67.31 78.74)
 		(diameter 0)
@@
 	(wire
 		(pts
-			(xy 252.73 92.71) (xy 252.73 118.11)
+			(xy 172.72 77.47) (xy 147.32 77.47)
 		)
 		(stroke
@@
 	(wire
 		(pts
-			(xy 172.72 77.47) (xy 147.32 77.47)
+			(xy 129.54 134.62) (xy 147.32 134.62)
 		)
 		(stroke
@@
 	(wire
 		(pts
-			(xy 129.54 134.62) (xy 147.32 134.62)
+			(xy 59.69 63.5) (xy 52.07 63.5)
 		)
 		(stroke
@@
 	(wire
 		(pts
-			(xy 59.69 63.5) (xy 52.07 63.5)
+			(xy 76.2 113.03) (xy 78.74 113.03)
 		)
 		(stroke
@@
 	(wire
 		(pts
-			(xy 76.2 113.03) (xy 78.74 113.03)
+			(xy 101.6 90.17) (xy 106.68 90.17)
 		)
 		(stroke
@@
 	(wire
 		(pts
-			(xy 101.6 90.17) (xy 106.68 90.17)
+			(xy 78.74 113.03) (xy 78.74 134.62)
 		)
 		(stroke
@@
 	(wire
 		(pts
-			(xy 78.74 113.03) (xy 78.74 134.62)
+			(xy 49.53 163.83) (xy 69.85 163.83)
 		)
 		(stroke
@@
 	(wire
 		(pts
-			(xy 49.53 163.83) (xy 69.85 163.83)
+			(xy 180.34 140.97) (xy 180.34 144.78)
 		)
 		(stroke
@@
 	(wire
 		(pts
-			(xy 222.25 118.11) (xy 222.25 120.65)
+			(xy 222.25 116.84) (xy 222.25 120.65)
 		)
 		(stroke
@@
 	(wire
 		(pts
-			(xy 222.25 116.84) (xy 222.25 118.11)
+			(xy 60.96 82.55) (xy 60.96 106.68)
 		)
 		(stroke
@@
 	(wire
 		(pts
-			(xy 60.96 82.55) (xy 60.96 106.68)
+			(xy 252.73 92.71) (xy 252.73 140.97)
 		)
 		(stroke
@@
 	(wire
 		(pts
-			(xy 91.44 134.62) (xy 91.44 137.16)
-		)
-		(stroke
-			(width 0)
-			(type default)
-		)
-	)
-	(wire
-		(pts
 			(xy 64.77 78.74) (xy 67.31 78.74)
 		)
@@
 	(wire
 		(pts
+			(xy 252.73 140.97) (xy 180.34 140.97)
+		)
+		(stroke
+			(width 0)
+			(type default)
+		)
+	)
+	(wire
+		(pts
 			(xy 31.75 163.83) (xy 46.99 163.83)
 		)
@@
 	(wire
 		(pts
-			(xy 180.34 128.27) (xy 180.34 144.78)
+			(xy 180.34 128.27) (xy 180.34 140.97)
 		)
 		(stroke
@@
 	(wire
 		(pts
-			(xy 90.17 137.16) (xy 90.17 179.07)
+			(xy 91.44 134.62) (xy 91.44 179.07)
 		)
 		(stroke
@@
 	(wire
 		(pts
-			(xy 90.17 137.16) (xy 91.44 137.16)
-		)
-		(stroke
-			(width 0)
-			(type default)
-		)
-	)
-	(wire
-		(pts
 			(xy 111.76 104.14) (xy 101.6 104.14)
 		)
@@
 	(wire
 		(pts
-			(xy 252.73 118.11) (xy 222.25 118.11)
-		)
-		(stroke
-			(width 0)
-			(type default)
-		)
-	)
-	(wire
-		(pts
 			(xy 29.21 39.37) (xy 30.48 39.37)
 		)
@@
 	)
 	(symbol
+		(lib_id "Diode:SMAJ5.0A")
+		(at 66.04 130.81 270)
+		(unit 1)
+		(body_style 1)
+		(exclude_from_sim no)
+		(in_bom yes)
+		(on_board yes)
+		(in_pos_files yes)
+		(dnp no)
+		(fields_autoplaced yes)
+		(property "Reference" "D3"
+			(at 68.58 129.5399 90)
+			(show_name no)
+			(do_not_autoplace no)
+			(effects
+				(font
+					(size 1.27 1.27)
+				)
+				(justify left)
+			)
+		)
+		(property "Value" "SMAJ5.0A"
+			(at 68.58 132.0799 90)
+			(show_name no)
+			(do_not_autoplace no)
+			(effects
+				(font
+					(size 1.27 1.27)
+				)
+				(justify left)
+			)
+		)
+		(property "Footprint" "Diode_SMD:D_SMA"
+			(at 60.96 130.81 0)
+			(hide yes)
+			(show_name no)
+			(do_not_autoplace no)
+			(effects
+				(font
+					(size 1.27 1.27)
+				)
+			)
+		)
+		(property "Datasheet" "https://www.littelfuse.com/media?resourcetype=datasheets&itemid=75e32973-b177-4ee3-a0ff-cedaf1abdb93&filename=smaj-datasheet"
+			(at 66.04 129.54 0)
+			(hide yes)
+			(show_name no)
+			(do_not_autoplace no)
+			(effects
+				(font
+					(size 1.27 1.27)
+				)
+			)
+		)
+		(property "Description" "400W unidirectional Transient Voltage Suppressor, 5.0Vr, SMA(DO-214AC)"
+			(at 66.04 130.81 0)
+			(hide yes)
+			(show_name no)
+			(do_not_autoplace no)
+			(effects
+				(font
+					(size 1.27 1.27)
+				)
+			)
+		)
+		(pin "2"
+		)
+		(pin "1"
+		)
+		(instances
+			(project "tracker_v4"
+				(path "/0704e846-b6bf-4206-baa8-1088b529855e/c73a9412-a8df-45fb-8b45-856a5aea081b"
+					(reference "D3")
+					(unit 1)
+				)
+			)
+		)
+	)
+	(symbol
 		(lib_id "Device:C")
 		(at 55.88 130.81 0)
@@
 	(symbol
 		(lib_id "power:GND")
-		(at 90.17 179.07 0)
+		(at 91.44 179.07 0)
 		(unit 1)
 		(body_style 1)
@@
 		(dnp no)
 		(property "Reference" "#PWR09"
-			(at 90.17 185.42 0)
+			(at 91.44 185.42 0)
 			(hide yes)
 			(show_name no)
@@
 		)
 		(property "Value" "GND"
-			(at 90.424 183.134 0)
+			(at 91.694 183.134 0)
 			(show_name no)
 			(do_not_autoplace no)
@@
 		)
 		(property "Footprint" ""
-			(at 90.17 179.07 0)
+			(at 91.44 179.07 0)
 			(hide yes)
 			(show_name no)
@@
 		)
 		(property "Datasheet" ""
-			(at 90.17 179.07 0)
+			(at 91.44 179.07 0)
 			(hide yes)
 			(show_name no)
@@
 		)
 		(property "Description" "Power symbol creates a global label with name \"GND\" , ground"
-			(at 90.17 179.07 0)
+			(at 91.44 179.07 0)
 			(hide yes)
 			(show_name no)
@@
 					(unit 1)
 				)
-			)
-		)
-	)
-	(symbol
-		(lib_id "Device:D")
-		(at 66.04 130.81 270)
-		(unit 1)
-		(body_style 1)
-		(exclude_from_sim no)
-		(in_bom yes)
-		(on_board yes)
-		(in_pos_files yes)
-		(dnp no)
-		(fields_autoplaced yes)
-		(property "Reference" "D5"
-			(at 68.58 129.5399 90)
-			(show_name no)
-			(do_not_autoplace no)
-			(effects
-				(font
-					(size 1.27 1.27)
-				)
-				(justify left)
-			)
-		)
-		(property "Value" "DO-214AC"
-			(at 68.58 132.0799 90)
-			(show_name no)
-			(do_not_autoplace no)
-			(effects
-				(font
-					(size 1.27 1.27)
-				)
-				(justify left)
-			)
-		)
-		(property "Footprint" "Diode_SMD:D_SMA"
-			(at 66.04 130.81 0)
-			(hide yes)
-			(show_name no)
-			(do_not_autoplace no)
-			(effects
-				(font
-					(size 1.27 1.27)
-				)
-			)
-		)
-		(property "Datasheet" "DO-214AC"
-			(at 66.04 130.81 0)
-			(hide yes)
-			(show_name no)
-			(do_not_autoplace no)
-			(effects
-				(font
-					(size 1.27 1.27)
-				)
-			)
-		)
-		(property "Description" "Diode"
-			(at 66.04 130.81 0)
-			(hide yes)
-			(show_name no)
-			(do_not_autoplace no)
-			(effects
-				(font
-					(size 1.27 1.27)
-				)
-			)
-		)
-		(property "Sim.Device" "D"
-			(at 66.04 130.81 0)
-			(hide yes)
-			(show_name no)
-			(do_not_autoplace no)
-			(effects
-				(font
-					(size 1.27 1.27)
-				)
-			)
-		)
-		(property "Sim.Pins" "1=K 2=A"
-			(at 66.04 130.81 0)
-			(hide yes)
-			(show_name no)
-			(do_not_autoplace no)
-			(effects
-				(font
-					(size 1.27 1.27)
-				)
-			)
-		)
-		(pin "2"
-		)
-		(pin "1"
-		)
-		(instances
-			(project "tracker_v4"
-				(path "/0704e846-b6bf-4206-baa8-1088b529855e/c73a9412-a8df-45fb-8b45-856a5aea081b"
-					(reference "D5")
-					(unit 1)
-				)

Commit message: jkd
Parts:
- removed U5: TP4056-42-ESOP8, Package_SO:SOIC-8-1EP_3.9x4.9mm_P1.27mm_EP2.41x3.3mm_ThermalVias, symbol Battery_Management:TP4056-42-ESOP8
- added C15: 4.7u, Capacitor_SMD:C_0805_2012Metric, symbol Device:C
- added R19: 2.1k, Resistor_SMD:R_0603_1608Metric, symbol Device:R
- added R20: 47k, symbol Device:R
- added R21: 10k, Resistor_SMD:R_0603_1608Metric, symbol Device:R
- added U8: BQ24072RGT, Package_DFN_QFN:VQFN-16-1EP_3x3mm_P0.5mm_EP1.6x1.6mm, symbol Battery_Management:BQ24072RGT
- C5: value 10u -> 4.7u
- R4: value 3.0k -> 1.5k
Connections:
- net BAT+: now also U8.2 (BAT), U8.3 (BAT)
- net GND: now also C15.1, R19.2, R20.2, R21.2, U8.15 (TD), U8.17 (VSS), U8.4 (~{CE}), U8.5 (EN2), U8.8 (VSS)
- net USB_VBUS: now also U8.13 (IN), U8.6 (EN1)
- net at D2.1 (K): now also U8.7 (~{PGOOD})
- net at R4.1: now also U8.12 (ILIM)
- net at D1.1 (K): now also U8.9 (~{CHG})
- new net: R20.1, U8.14 (TMR)
- new net: R21.1, U8.1 (TS)
- new net: R19.1, U8.16 (ISET)
- new net POWER_OUT: C15.2, U8.10 (OUT), U8.11 (OUT)
Other:
- moved on the sheet: D1, D2, R10, R8, TP7

Commit message: newer version
Parts:
- BT1: footprint Connector_JST:JST_PH_S2B-PH-K_1x02_P2.00mm_Horizontal -> Connector_JST:JST_SH_SM02B-SRSS-TB_1x02-1MP_P1.00mm_Horizontal
- C15: value 4.7u -> 10u
- C6: footprint Capacitor_SMD:C_0603_1608Metric -> Capacitor_SMD:C_0805_2012Metric
- R20: footprint (none) -> Resistor_SMD:R_0603_1608Metric
- R7: value 100 -> 500
- R9: value 1k -> 1.5k
Changed lines of the file:
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@@
 			)
 		)
-		(property "Value" "1k"
+		(property "Value" "1.5k"
 			(at 255.27 90.1699 0)
 			(show_name no)
@@
 			)
 		)
-		(property "Value" "100"
+		(property "Value" "500"
 			(at 140.97 77.47 90)
 			(show_name no)
@@
 			)
 		)
-		(property "Footprint" ""
+		(property "Footprint" "Resistor_SMD:R_0603_1608Metric"
 			(at 79.502 153.67 90)
 			(hide yes)
@@
 			)
 		)
-		(property "Value" "4.7u"
+		(property "Value" "10u"
 			(at 97.79 73.6599 0)
 			(show_name no)
@@
 			)
 		)
-		(property "Footprint" "Capacitor_SMD:C_0603_1608Metric"
+		(property "Footprint" "Capacitor_SMD:C_0805_2012Metric"
 			(at 110.7948 104.14 0)
 			(hide yes)
@@
 			)
 		)
-		(property "Footprint" "Connector_JST:JST_PH_S2B-PH-K_1x02_P2.00mm_Horizontal"
+		(property "Footprint" "Connector_JST:JST_SH_SM02B-SRSS-TB_1x02-1MP_P1.00mm_Horizontal"
 			(at 129.54 124.206 90)
 			(hide yes)

Commit message: b
Parts:
- BT1: footprint Connector_JST:JST_SH_SM02B-SRSS-TB_1x02-1MP_P1.00mm_Horizontal -> Connector_JST:JST_PH_S2B-PH-K_1x02_P2.00mm_Horizontal
- R7: value 500 -> 499
Changed lines of the file:
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@@
 			)
 		)
-		(property "Value" "500"
+		(property "Value" "499"
 			(at 140.97 77.47 90)
 			(show_name no)
@@
 			)
 		)
-		(property "Footprint" "Connector_JST:JST_SH_SM02B-SRSS-TB_1x02-1MP_P1.00mm_Horizontal"
+		(property "Footprint" "Connector_JST:JST_PH_S2B-PH-K_1x02_P2.00mm_Horizontal"
 			(at 129.54 124.206 90)
 			(hide yes)
