File: tracker_v4/tracker_v4.kicad_pcb (KiCad board)
At the start: 4 copper layers, 63.2 x 26 mm, 53 parts, among them IC1 RT9080-33GJ5, J1 USB_C_Receptacle_USB2.0_16P, Q1 DMG9926UDM-7, U1 ESP32-C6-MINI-1-N4, U2 LIS3DH, U3 DW01A, U4 INA226AIDGSR, U5 TP4056-42-ESOP8, U6 USBLC6-2SC6, U7 TPS3899DL01DSER

Commit message: newer version
Parts:
- removed IC1: RT9080-33GJ5, RT9080-33GJ5:SOT94P280X100-5N
- added C14: 22u, Capacitor_SMD:C_1206_3216Metric, F.Cu at (132.9, 122.1)
- added C15: 10u, Capacitor_SMD:C_0805_2012Metric, F.Cu at (142.2, 112.8)
- added C16: 10u, Capacitor_SMD:C_0805_2012Metric, F.Cu at (145.0, 121.9)
- added C17: 100n, Capacitor_SMD:C_0603_1608Metric, F.Cu at (143.9, 119.5)
- added C18: 10u, Capacitor_SMD:C_0805_2012Metric, F.Cu at (141.4, 117.4)
- added L1: 1.5u, Inductor_SMD:L_Coilcraft_XxL4020, F.Cu at (137.5, 115.0)
- added R17: 1M, Resistor_SMD:R_0603_1608Metric, F.Cu at (141.3, 121.3)
- added R18: 180k, Resistor_SMD:R_0603_1608Metric, F.Cu at (143.9, 117.7)
- added R19: 2.1k, Resistor_SMD:R_0603_1608Metric, F.Cu at (152.2, 120.7)
- added R20: 47k, Resistor_SMD:R_0603_1608Metric, F.Cu at (148.8, 122.1)
- added R21: 10k, Resistor_SMD:R_0603_1608Metric, F.Cu at (153.7, 113.2)
- added R22: 10k, Resistor_SMD:R_0603_1608Metric, F.Cu at (120.0, 122.1)
- added R23: 10M, Resistor_SMD:R_0603_1608Metric, F.Cu at (134.1, 120.2)
- added U8: BQ24072RGT, Package_DFN_QFN:VQFN-16-1EP_3x3mm_P0.5mm_EP1.6x1.6mm, F.Cu at (148.6, 115.1)
- BT1: footprint Connector_JST:JST_PH_S2B-PH-K_1x02_P2.00mm_Horizontal -> Connector_JST:JST_SH_SM02B-SRSS-TB_1x02-1MP_P1.00mm_Horizontal
- C5: value 10u -> 4.7u
- C6: footprint Capacitor_SMD:C_0603_1608Metric -> Capacitor_SMD:C_0805_2012Metric
- C8: value 10u -> 22u; footprint Capacitor_SMD:C_0805_2012Metric -> Capacitor_SMD:C_1206_3216Metric
- R14: value 1.27M -> 1000k
- R15: value 226k -> 200k
- R4: value 3.0k -> 1.5k
- R7: value 100 -> 500
- R9: value 1k -> 1.5k
- U5: value TP4056-42-ESOP8 -> TPS63020; footprint Package_SO:SOIC-8-1EP_3.9x4.9mm_P1.27mm_EP2.41x3.3mm_ThermalVias -> TPS63020:TPS63020
- moved BT1 18.9 mm to (154.0, 102.0), turned to 90 degrees
- moved U5 10.6 mm to (138.5, 120.0), turned to -90 degrees
- moved TP7 1.60 mm to (158.6, 106.6)
- moved D3 1.31 mm to (163.0, 107.4), turned to 0 degrees
- moved C10 0.89 mm to (124.8, 107.1), turned to 180 degrees
- turned C6 to 180 degrees
Connections:
- BT1 pad 1: /Charging_and_Battery/BAT+ -> BAT+
- C6 pad 2: /Charging_and_Battery/BAT+ -> BAT+
- C8 pad 1: SHUNT_OUTPUT -> 3v3
- R1 pad 1: /Charging_and_Battery/BAT+ -> POWER_OUT
- R16 pad 2: LDO_EN -> BUCK_EN
- R4 pad 1: Net-(U5-PROG) -> Net-(U8-ILIM)
- R7 pad 1: /Charging_and_Battery/BAT+ -> BAT+
- TP8 pad 1: /Charging_and_Battery/BAT+ -> BAT+
- U1 pad 9: unconnected-(U1-IO4-Pad9) -> BUCK_SYNC
- U4 pad 10: /Charging_and_Battery/BAT+ -> POWER_OUT
- U7 pad 6: LDO_EN -> BUCK_EN
Routing:
- net BAT+: track 0.00 -> 51.4 mm, vias 0 -> 6
- net /Charging_and_Battery/BAT+: track 48.5 -> 0.00 mm, vias 4 -> 0
- net SHUNT_OUTPUT: track 30.8 -> 70.6 mm, vias 0 -> 3
- net POWER_OUT: track 0.00 -> 32.1 mm, vias 0 -> 4
- net BUCK_EN: track 0.00 -> 26.8 mm, vias 0 -> 3
- net BUCK_SYNC: track 0.00 -> 26.1 mm, vias 0 -> 4
- net GND: track 144.4 -> 165.4 mm, vias 74 -> 72
- net 3v3: track 93.2 -> 111.9 mm, vias 16 -> 17
- net /Charging_and_Battery/BAT-: track 8.31 -> 19.4 mm, vias 0 -> 2
- net UVLO_SENSE: track 10.7 -> 21.7 mm, vias 0 -> 2
- net LDO_EN: track 9.22 -> 0.00 mm, vias 2 -> 0
- net Net-(U5-FB): track 0.00 -> 9.04 mm, vias 0 -> 2
- net USB_VBUS: track 61.0 -> 68.9 mm, vias 5 -> 6
- net Net-(U8-TMR): track 0.00 -> 7.02 mm, vias 0 -> 2
- net Net-(U8-ILIM): track 0.00 -> 6.85 mm, vias 0 -> 2
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
Commit message: b
Parts:
- removed the C9 at (129.5, 109.0)
- added C9: 22u, Capacitor_SMD:C_1206_3216Metric, F.Cu at (141.1, 116.8)
- added C9: 22u, Capacitor_SMD:C_1206_3216Metric, F.Cu at (137.5, 110.1)
- BT1: footprint Connector_JST:JST_SH_SM02B-SRSS-TB_1x02-1MP_P1.00mm_Horizontal -> Connector_JST:JST_PH_S2B-PH-K_1x02_P2.00mm_Horizontal
- R7: value 500 -> 499
- moved C8 19.8 mm to (142.2, 113.3), turned to 0 degrees
- moved C6 16.1 mm to (153.5, 112.2)
- moved C17 14.1 mm to (129.9, 121.3), turned to 0 degrees
- moved C16 12.6 mm to (132.4, 121.3), turned to 90 degrees
- moved C10 12.4 mm to (134.4, 114.9), turned to 90 degrees
- moved R23 12.4 mm to (125.3, 111.5)
- moved C14 11.5 mm to (144.3, 120.8), turned to -90 degrees
- moved C5 8.07 mm to (144.0, 116.2), turned to 180 degrees
- moved C18 7.74 mm to (134.4, 120.7), turned to 90 degrees
- moved C15 4.74 mm to (146.2, 110.2)
- moved R19 3.08 mm to (151.5, 117.7), turned to 0 degrees
- moved R5 2.72 mm to (168.0, 118.5), turned to 90 degrees
- moved BT1 1.97 mm to (152.3, 103.0)
- moved R6 1.96 mm to (154.8, 117.8), turned to 90 degrees
- moved R21 1.50 mm to (153.4, 114.7), turned to 90 degrees
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Routing:
- net BAT+: track 51.4 -> 40.4 mm, vias 6 -> 5
- net 3v3: track 111.9 -> 122.7 mm
- net USB_VBUS: track 68.9 -> 58.9 mm, vias 6 -> 5
- net Net-(J1-CC2): track 9.47 -> 5.87 mm
- net BUCK_SYNC: track 26.1 -> 28.8 mm
- net Net-(U8-ISET): track 5.00 -> 2.40 mm, vias 2 -> 0
- net UVLO_SENSE: track 21.7 -> 19.3 mm, vias 2 -> 3
- net POWER_OUT: track 32.1 -> 34.4 mm
- net /Charging_and_Battery/BAT-: track 19.4 -> 17.4 mm
- net USB_DP: track 59.3 -> 61.4 mm
- net BUCK_EN: track 26.8 -> 28.3 mm
- net Net-(U8-ILIM): track 6.85 -> 5.52 mm
- net Net-(J1-CC1): track 9.74 -> 8.51 mm
- net SHUNT_OUTPUT: track 70.6 -> 69.5 mm, vias 3 -> 4
- net GND: track 165.4 -> 166.4 mm, vias 72 -> 66
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Other:
- board size 63.2 x 26 mm -> 62.5 x 26.3 mm
